File: KiCad/CC1101_RPi/CC1101_RPi.kicad_pcb (KiCad board)
At the start: 2 copper layers, 85 x 56 mm, 150 parts, among them J1001 SMA_433, J2001 SMA_433, J3001 SMA_868, J4001 SMA_868, J6001 Raspberry_Pi_4, Q1001 2N7002, Q1002 2N7002, Q2001 2N7002, Q2002 2N7002, Q3001 2N7002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

Commit message: Production to JLCPCB
Routing:
- net +3.3V: track 332.4 -> 330.9 mm
- net +5V: track 121.3 -> 120.3 mm
- net GND: track 239.4 -> 238.5 mm, vias 80 -> 81
- net /SCLK_2: track 90.0 -> 89.2 mm
- net /MOSI_1: track 74.3 -> 73.5 mm
- net Net-(J1001-In): track 18.5 -> 17.8 mm
- net /GDO2_4: track 35.1 -> 34.4 mm
